File: videoslot/videoslot.sch (KiCad schematic (older format))
At the start: 9 parts, among them P1 CONN_02X08, U1 74LVC8T245, U2 74LVC8T245

Commit message: VA2000CX corrections for PCB batch 1
Parts:
- removed P1: CONN_02X08, Pin_Headers:Pin_Header_Straight_2x08, symbol CONN_02X08
- added P1: UPLINK, Pin_Headers:Pin_Header_Straight_2x18_Pitch2.54mm, symbol CONN_02X18
- added P2: PMOD1, Pin_Headers:Pin_Header_Angled_1x06_Pitch2.54mm, symbol CONN_01X06
- added P3: PMOD2, Pin_Headers:Pin_Header_Angled_2x06_Pitch2.54mm, symbol CONN_02X06
- renumbered C4 to C3, C5 to C4, C3 to CN1, C6 to CN2
Connections:
- net labels added: +3.3V, +5V, HS, VS, b0, b1, b2, b3, g0, g1, g2, g3, r0, r1, r2, r3
- wire segments 114 -> 165
Other:
- moved on the sheet: C1, C2, C3, C4, CN2, U1, U2

Commit message: WIP 1.5b firmware, gfx drivers; mntmode, va2000cx initial commits
Parts:
- CN1: symbol CN451 -> CN451-RESCUE-videoslot
Connections:
- wire segments 165 -> 166
