File: videoslot/videoslot.sch (KiCad schematic (older format))
At the start: 11 parts, among them CN1 CN451/203, CN2 CN452/207, P1 UPLINK, P2 PMOD1, P3 PMOD2, U1 74LVC8T245, U2 74LVC8T245

Commit message: Update of schematics and project files to KiCad 5.1
Parts:
- C1, C2, C3, C4: symbol C_Small -> videoslot-rescue:C_Small
- CN1: symbol CN451-RESCUE-videoslot -> videoslot-rescue:CN451-RESCUE-videoslot
- CN2: symbol CN452 -> videoslot-rescue:CN452
- P1: symbol CONN_02X18 -> videoslot-rescue:CONN_02X18
- P2: symbol CONN_01X06 -> videoslot-rescue:CONN_01X06
- P3: symbol CONN_02X06 -> videoslot-rescue:CONN_02X06
- U1, U2: symbol 74LVC8T245 -> videoslot-rescue:74LVC8T245
Changed lines of the file:
@@
-EESchema Schematic File Version 2
-LIBS:power
-LIBS:device
-LIBS:transistors
-LIBS:conn
-LIBS:linear
-LIBS:xilinx
-LIBS:regul
-LIBS:74xx
-LIBS:cmos4000
-LIBS:adc-dac
-LIBS:memory
-LIBS:microcontrollers
-LIBS:dsp
-LIBS:microchip
-LIBS:analog_switches
-LIBS:motorola
-LIBS:texas
-LIBS:intel
-LIBS:audio
-LIBS:interface
-LIBS:digital-audio
-LIBS:philips
-LIBS:display
-LIBS:cypress
-LIBS:siliconi
-LIBS:opto
-LIBS:atmel
-LIBS:contrib
-LIBS:valves
-LIBS:mntamiga
-LIBS:voltrans
-LIBS:74lvc8t245
-EELAYER 25 0
+EESchema Schematic File Version 4
+LIBS:videoslot-cache
+EELAYER 29 0
 EELAYER END
 $Descr A4 11693 8268
@@
 $EndDescr
 $Comp
-L CN451-RESCUE-videoslot CN1
+L videoslot-rescue:CN451-RESCUE-videoslot CN1
 U 1 1 579D05C5
 P 4350 4550
@@
 $EndComp
 $Comp
-L CN452 CN2
+L videoslot-rescue:CN452 CN2
 U 1 1 579D07DC
 P 7400 4550
@@
 $EndComp
 $Comp
-L 74LVC8T245 U1
+L videoslot-rescue:74LVC8T245 U1
 U 1 1 579D1430
 P 3100 4200
@@
 $EndComp
 $Comp
-L 74LVC8T245 U2
+L videoslot-rescue:74LVC8T245 U2
 U 1 1 579D17F7
 P 6350 3400
@@
 $EndComp
 $Comp
-L C_Small C1
+L videoslot-rescue:C_Small C1
 U 1 1 579D32F5
 P 2800 3150
@@
 $EndComp
 $Comp
-L C_Small C2
+L videoslot-rescue:C_Small C2
 U 1 1 579D33BE
 P 3600 3150
@@
 $EndComp
 $Comp
-L C_Small C3
+L videoslot-rescue:C_Small C3
 U 1 1 579D340B
 P 6100 2450
@@
 $EndComp
 $Comp
-L C_Small C4
+L videoslot-rescue:C_Small C4
 U 1 1 579D3462
 P 6650 2450
@@
 $EndComp
 $Comp
-L GND #PWR01
+L videoslot-rescue:GND #PWR01
 U 1 1 579D3499
 P 6100 2350
@@
 $EndComp
 $Comp
-L GND #PWR02
+L videoslot-rescue:GND #PWR02
 U 1 1 579D34BF
 P 6650 2350
@@
 $EndComp
 $Comp
-L GND #PWR03
+L videoslot-rescue:GND #PWR03
 U 1 1 579D352D
 P 2800 3050
@@
 $EndComp
 $Comp
-L GND #PWR04
+L videoslot-rescue:GND #PWR04
 U 1 1 579D3553
 P 3600 3050
@@
 $EndComp
 $Comp
-L GND #PWR05
+L videoslot-rescue:GND #PWR05
 U 1 1 579D359D
 P 3750 4650
@@
 $EndComp
 $Comp
-L GND #PWR06
+L videoslot-rescue:GND #PWR06
 U 1 1 579D35C3
 P 2650 4800
@@
 $EndComp
 $Comp
-L GND #PWR07
+L videoslot-rescue:GND #PWR07
 U 1 1 579D360D
 P 6750 5150
@@
 $EndComp
 $Comp
-L GND #PWR08
+L videoslot-rescue:GND #PWR08
 U 1 1 579D3633
 P 5900 3900
@@
 $EndComp
 $Comp
-L CONN_02X18 P1
+L videoslot-rescue:CONN_02X18 P1
 U 1 1 58BC318E
 P 3800 1600
@@
 VS
 $Comp
-L GND #PWR09
+L videoslot-rescue:GND #PWR09
 U 1 1 58BC4F1C
 P 3350 1350
@@
 $EndComp
 $Comp
-L GND #PWR010
+L videoslot-rescue:GND #PWR010
 U 1 1 58BC4F54
 P 4150 1350
@@
 $EndComp
 $Comp
-L GND #PWR011
+L videoslot-rescue:GND #PWR011
 U 1 1 58BC4F8C
 P 4150 1850
@@
 $EndComp
 $Comp
-L +5V #PWR012
+L videoslot-rescue:+5V #PWR012
 U 1 1 58BC54C4
 P 4650 1350
@@
 $EndComp
 $Comp
-L +5V #PWR013
+L videoslot-rescue:+5V #PWR013
 U 1 1 58BC54F3
 P 4650 1850
@@
 $EndComp
 $Comp
-L GND #PWR014
+L videoslot-rescue:GND #PWR014
 U 1 1 58BC594B
 P 4350 5550
@@
 $EndComp
 $Comp
-L GND #PWR015
+L videoslot-rescue:GND #PWR015
 U 1 1 58BC597A
 P 4350 5150
@@
 $EndComp
 $Comp
-L GND #PWR016
+L videoslot-rescue:GND #PWR016
 U 1 1 58BC5ABD
 P 4350 5750
@@
 $EndComp
 $Comp
-L GND #PWR017
+L videoslot-rescue:GND #PWR017
 U 1 1 58BC5DD6
 P 7400 2600
@@
 $EndComp
 $Comp
-L +3.3V #PWR018
+L videoslot-rescue:+3.3V #PWR018
 U 1 1 58BC5FFD
 P 2950 1350
@@
 $EndComp
 $Comp
-L +3.3V #PWR019
+L videoslot-rescue:+3.3V #PWR019
 U 1 1 58BC6023
 P 2950 1850
@@
 $EndComp
 $Comp
-L +3.3V #PWR020
+L videoslot-rescue:+3.3V #PWR020
 U 1 1 58BC619F
 P 5950 2550
@@
 $EndComp
 $Comp
-L +3.3V #PWR021
+L videoslot-rescue:+3.3V #PWR021
 U 1 1 58BC6512
 P 2550 3100
@@
 $EndComp
 $Comp
-L CONN_01X06 P2
+L videoslot-rescue:CONN_01X06 P2
 U 1 1 58BC6655
 P 6250 650
@@
 $EndComp
 $Comp
-L CONN_02X06 P3
+L videoslot-rescue:CONN_02X06 P3
 U 1 1 58BC6734
 P 7450 1600
@@
 $EndComp
 $Comp
-L GND #PWR022
+L videoslot-rescue:GND #PWR022
 U 1 1 58BC7FAC
 P 6400 900
@@
 $EndComp
 $Comp
-L GND #PWR023
+L videoslot-rescue:GND #PWR023
 U 1 1 58BC80A4
 P 7600 1350
@@
 $EndComp
 $Comp
-L GND #PWR024
+L videoslot-rescue:GND #PWR024
 U 1 1 58BC80E4
 P 7600 1850
@@
 $EndComp
 $Comp
-L +3.3V #PWR025
+L videoslot-rescue:+3.3V #PWR025
 U 1 1 58BC810E
 P 6500 900
@@
 $EndComp
 $Comp
-L +3.3V #PWR026
+L videoslot-rescue:+3.3V #PWR026
 U 1 1 58BC8143
 P 7700 1350
@@
 $EndComp
 $Comp
-L +3.3V #PWR027
+L videoslot-rescue:+3.3V #PWR027
 U 1 1 58BC8178
 P 7700 1850
@@
 $EndComp
 $Comp
-L +5V #PWR028
+L videoslot-rescue:+5V #PWR028
 U 1 1 58BC9DB5
 P 3650 3400
@@
 $EndComp
 $Comp
-L +5V #PWR029
+L videoslot-rescue:+5V #PWR029
 U 1 1 58BC9DEA
 P 6900 2700
@@
 $EndComp
 $Comp
-L GND #PWR030
+L videoslot-rescue:GND #PWR030
 U 1 1 58BDE7DB
 P 3750 1350
@@
 $EndComp
 $Comp
-L GND #PWR031
+L videoslot-rescue:GND #PWR031
 U 1 1 58BDE86A
 P 3750 1850
@@
 $EndComp
 $Comp
-L GND #PWR032
+L videoslot-rescue:GND #PWR032
 U 1 1 58BDE8EE
 P 3350 1850
@@
 	3500 4150 4350 4150
 Wire Wire Line
-	3500 3550 4150 3550
+	3500 3550 3600 3550
 Wire Wire Line
 	3600 3650 3500 3650
 Wire Wire Line
-	3600 3250 3600 3650
+	3600 3250 3600 3400
 Connection ~ 3600 3550
 Wire Wire Line
@@
 	6750 5150 7400 5150
 Wire Wire Line
-	6750 3850 6750 5150
-Wire Wire Line
-	6750 2750 6750 2850
-Wire Wire Line
-	6850 2550 6850 2800
+	6750 3850 6750 3900
+Wire Wire Line
+	6750 2750 6750 2800
+Wire Wire Line
+	6850 2550 6850 2700
 Wire Wire Line
 	6850 2800 6750 2800
@@
 	2550 3100 2550 3550
 Wire Wire Line
-	2550 3550 2700 3550
+	2550 3550 2650 3550
 Wire Wire Line
 	5600 2950 5950 2950
@@
 	2700 3650 2650 3650
 Wire Wire Line
-	2650 3650 2650 4800
+	2650 3650 2650 4550
 Wire Wire Line
 	5900 3850 5950 3850
 Wire Wire Line
-	5900 2850 5900 3900
+	5900 2850 5900 3750
 Connection ~ 5900 3750
 Wire Wire Line
@@
 	3500 3750 3600 3750
 Wire Wire Line
-	3600 3750 3600 6150
-Wire Wire Line
-	3500 4650 3750 4650
+	3600 3750 3600 4650
+Wire Wire Line
+	3500 4650 3600 4650
 Connection ~ 3600 4650
 Wire Wire Line
@@
 	5250 2450 5250 3650
 Wire Wire Line
-	7400 2600 7400 3150
+	7400 2600 7400 2750
 Connection ~ 7400 2950
 Connection ~ 7400 2750
@@
 Wire Wire Line
 	4150 4850 4350 4850
+Wire Wire Line
+	3600 3550 4150 3550
+Wire Wire Line
+	3600 3550 3600 3650
+Wire Wire Line
+	6750 2800 6750 2850
+Wire Wire Line
+	5900 3750 5900 3850
+Wire Wire Line
+	2650 4550 2650 4650
+Wire Wire Line
+	3600 4650 3600 6150
+Wire Wire Line
+	3600 4650 3750 4650
+Wire Wire Line
+	6750 3900 6750 5150
+Wire Wire Line
+	5900 3850 5900 3900
+Wire Wire Line
+	2650 3550 2700 3550
+Wire Wire Line
+	7400 2950 7400 3150
+Wire Wire Line
+	7400 2750 7400 2950
+Wire Wire Line
+	2650 4650 2650 4800
+Wire Wire Line
+	6850 2700 6850 2800
+Wire Wire Line
+	3600 3400 3600 3550
 $EndSCHEMATC
